File: Robotrace/Robotrace.kicad_sch (KiCad schematic)
At the start: 55 parts, among them J1 USB_C_Receptacle_USB2.0_16P, J10 Side_L, J11 LINE, J6 STDC14, J7 Conn_02x05_Odd_Even, J8 Conn_02x05_Odd_Even, J9 Side_R, Q5 BSS138, SW1 SW_DPDT_x2, U1 STM32F469VGTx, Y1 FA-238V 12.000000MHz

Commit message: 配線
Parts:
- removed SW1: SW_DPDT_x2, symbol Switch:SW_DPDT_x2
- added C37, C38, C39, C40: 0.1u, Capacitor_SMD:C_0603_1608Metric, symbol Device:C_Small
- added D10, D11, D8, D9: WS2812B, LED_SMD:LED_WS2812B-2020_PLCC4_2.0x2.0mm, symbol LED:WS2812B
- BZ1: footprint (none) -> Buzzer_Beeper:Buzzer_Murata_PKMCS0909E
- C1, C15, C16, C17, C18, C19, C20, C21, C24, C25, C26, C27, C28, C29, C30, C31, C32, C33, C34, C35, C36: footprint Capacitor_SMD:C_0402_1005Metric -> Capacitor_SMD:C_0603_1608Metric
- D3, D4, D5, D6: footprint (none) -> LED_SMD:LED_0603_1608Metric
- FB1, FB2: footprint (none) -> Capacitor_SMD:C_0603_1608Metric
- J10, J9: footprint (none) -> Connector_JST:JST_SH_SM03B-SRSS-TB_1x03-1MP_P1.00mm_Horizontal
- J11: footprint (none) -> 5051101892:CON_5051101892_MOL
- J6: footprint Connector_PinSocket_1.27mm:PinSocket_2x07_P1.27mm_Vertical -> Connector_PinHeader_1.27mm:PinHeader_2x07_P1.27mm_Vertical_SMD
- J7, J8: footprint (none) -> Connector_PinHeader_1.27mm:PinHeader_2x05_P1.27mm_Vertical
- Y1: value FA-238V 12.000000MHz -> 12MHz; footprint (none) -> Crystal:Crystal_SMD_3225-4Pin_3.2x2.5mm
Connections:
- net +5V: now also C37.1, C38.1, C39.1, C40.1, D10.1 (VDD), D11.1 (VDD), D8.1 (VDD), D9.1 (VDD)
- net GND: now also C37.2, C38.2, C39.2, C40.2, D10.3 (VSS), D11.3 (VSS), D8.3 (VSS), D9.3 (VSS)
- new net: D10.2 (DOUT), D11.4 (DIN)
- new net: D10.4 (DIN), D9.2 (DOUT)
- new net: D8.2 (DOUT), D9.4 (DIN)
- new net FLED: D8.4 (DIN)
Other:
- sheet DC-DC ports: added none; removed EN
