File: Robotrace/Robotrace.kicad_sch (KiCad schematic)
At the start: 62 parts, among them J1 USB_C_Receptacle_USB2.0_16P, J10 Side_L, J11 LINE, J6 STDC14, J7 Conn_02x05_Odd_Even, J8 Conn_02x05_Odd_Even, J9 Side_R, Q5 BSS138, U1 STM32F469VGTx, Y1 12MHz

Commit message: PWM/エンコーダ配線の復旧とIMU_INT1/INT2のMCU接続を追加
ユーザーのKiCad上での保存時に、PWM_A_L/B_L/A_R/B_RとEnc_A_L/B_L/A_R/B_RのMCU側配線(PA8,PB8,PB9,PC9,PB4,PB5,PC6,PC7)が失われていたため復旧。
あわせてIMU_INT1/INT2がMCUに未接続だった問題を修正(PD0->IMU_INT1, PD1->IMU_INT2)。既存のPA-PCポートが全て使用済みだったため、未使用のPD/PEポートがあることを確認しPD0/PD1を採用。

Co-Authored-By: Claude Sonnet 5 <noreply@anthropic.com>
Claude-Session: https://claude.ai/code/session_01781fWTRjWjmRZVNFFPgVZP
Connections:
- net Enc_A_L: now also U1.93 (PB4)
- net Enc_A_R: now also U1.66 (PC6)
- net Enc_B_L: now also U1.94 (PB5)
- net Enc_B_R: now also U1.67 (PC7)
- net IMU_INT1: now also U1.84 (PD0)
- net IMU_INT2: now also U1.85 (PD1)
- net PWM_A_L: now also U1.70 (PA8)
- net PWM_A_R: now also U1.99 (PB9)
- net PWM_B_L: now also U1.98 (PB8)
- net PWM_B_R: now also U1.69 (PC9)
Changed lines of the file:
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@@
+		)
+	)
+	(wire
+		(pts
+			(xy 149.86 80.01) (xy 152.4 80.01)
+		)
+		(stroke
+			(width 0)
+			(type default)
+		)
+	)
+	(label "PWM_A_L"
+		(at 152.4 80.01 0)
+		(effects
+			(font
+				(size 1.27 1.27)
+			)
+			(justify left bottom)
+		)
+	)
+	(wire
+		(pts
+			(xy 149.86 123.19) (xy 152.4 123.19)
+		)
+		(stroke
+			(width 0)
+			(type default)
+		)
+	)
+	(label "PWM_B_L"
+		(at 152.4 123.19 0)
+		(effects
+			(font
+				(size 1.27 1.27)
+			)
+			(justify left bottom)
+		)
+	)
+	(wire
+		(pts
+			(xy 149.86 125.73) (xy 152.4 125.73)
+		)
+		(stroke
+			(width 0)
+			(type default)
+		)
+	)
+	(label "PWM_A_R"
+		(at 152.4 125.73 0)
+		(effects
+			(font
+				(size 1.27 1.27)
+			)
+			(justify left bottom)
+		)
+	)
+	(wire
+		(pts
+			(xy 149.86 163.83) (xy 152.4 163.83)
+		)
+		(stroke
+			(width 0)
+			(type default)
+		)
+	)
+	(label "PWM_B_R"
+		(at 152.4 163.83 0)
+		(effects
+			(font
+				(size 1.27 1.27)
+			)
+			(justify left bottom)
+		)
+	)
+	(wire
+		(pts
+			(xy 149.86 113.03) (xy 152.4 113.03)
+		)
+		(stroke
+			(width 0)
+			(type default)
+		)
+	)
+	(label "Enc_A_L"
+		(at 152.4 113.03 0)
+		(effects
+			(font
+				(size 1.27 1.27)
+			)
+			(justify left bottom)
+		)
+	)
+	(wire
+		(pts
+			(xy 149.86 115.57) (xy 152.4 115.57)
+		)
+		(stroke
+			(width 0)
+			(type default)
+		)
+	)
+	(label "Enc_B_L"
+		(at 152.4 115.57 0)
+		(effects
+			(font
+				(size 1.27 1.27)
+			)
+			(justify left bottom)
+		)
+	)
+	(wire
+		(pts
+			(xy 149.86 156.21) (xy 152.4 156.21)
+		)
+		(stroke
+			(width 0)
+			(type default)
+		)
+	)
+	(label "Enc_A_R"
+		(at 152.4 156.21 0)
+		(effects
+			(font
+				(size 1.27 1.27)
+			)
+			(justify left bottom)
+		)
+	)
+	(wire
+		(pts
+			(xy 149.86 158.75) (xy 152.4 158.75)
+		)
+		(stroke
+			(width 0)
+			(type default)
+		)
+	)
+	(label "Enc_B_R"
+		(at 152.4 158.75 0)
+		(effects
+			(font
+				(size 1.27 1.27)
+			)
+			(justify left bottom)
+		)
+	)
+	(wire
+		(pts
+			(xy 77.47 128.27) (xy 83.82 128.27)
+		)
+		(stroke
+			(width 0)
+			(type default)
+		)
+	)
+	(label "IMU_INT1"
+		(at 77.47 128.27 0)
+		(effects
+			(font
+				(size 1.27 1.27)
+			)
+			(justify right bottom)
+		)
+	)
+	(wire
+		(pts
+			(xy 77.47 130.81) (xy 83.82 130.81)
+		)
+		(stroke
+			(width 0)
+			(type default)
+		)
+	)
+	(label "IMU_INT2"
+		(at 77.47 130.81 0)
+		(effects
+			(font
+				(size 1.27 1.27)
+			)
+			(justify right bottom)
 		)
 	)

Commit message: ピン配置を物理隣接性に基づき再編成(IMU/左右モーター群をクラスタ化)
STM32F469VGT6のLQFP100パッケージの物理ピン番号を調べ、関連信号が基板上で隣接するよう再配置した。

- IMUクラスタ: SPI(CS/CLK/MISO/MOSI = PB12-15, 物理ピン46-49)の直後にINT1/INT2(PD8/PD9, ピン50-51)を配置し、6本が連続。
- 左モーター群(TIM8): Enc_A_L/Enc_B_L/PWM_A_L/PWM_B_L = PC6/PC7/PC8/PC9(ピン66-69)で連続。エンコーダをCH1/CH2、PWMをCH3/CH4に割当。
- 右モーター群(TIM4): Enc_A_R/Enc_B_R/PWM_A_R/PWM_B_R = PB6/PB7/PB8/PB9(ピン95・96・98・99)で連続。
- 上記により押し出されたLED_3->PB4、SW_2->PB5に再配置。PA8は未使用化。

Co-Authored-By: Claude Sonnet 5 <noreply@anthropic.com>
Claude-Session: https://claude.ai/code/session_01781fWTRjWjmRZVNFFPgVZP
Connections:
- net Enc_A_L: now also U1.66 (PC6); no longer U1.93 (PB4)
- net Enc_A_R: now also U1.95 (PB6); no longer U1.66 (PC6)
- net Enc_B_L: now also U1.67 (PC7); no longer U1.94 (PB5)
- net Enc_B_R: now also U1.96 (PB7); no longer U1.67 (PC7)
- net IMU_INT1: now also U1.50 (PD8); no longer U1.84 (PD0)
- net IMU_INT2: now also U1.51 (PD9); no longer U1.85 (PD1)
- net LED_3: now also U1.93 (PB4); no longer U1.95 (PB6)
- net PWM_A_L: now also U1.68 (PC8); no longer U1.70 (PA8)
- net PWM_A_R: now also U1.98 (PB8); no longer U1.99 (PB9)
- net PWM_B_L: now also U1.69 (PC9); no longer U1.98 (PB8)
- net PWM_B_R: now also U1.99 (PB9); no longer U1.69 (PC9)
- net SW_2: now also U1.94 (PB5); no longer U1.68 (PC8)
Changed lines of the file:
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@@
 		)
 	)
-	(label "LED_3"
+	(label "Enc_A_R"
 		(at 152.4 118.11 0)
 		(effects
@@
 		)
 	)
-	(label "SW_2"
+	(label "PWM_A_L"
 		(at 152.4 161.29 0)
 		(effects
@@
 	(wire
 		(pts
-			(xy 149.86 80.01) (xy 152.4 80.01)
+			(xy 149.86 123.19) (xy 152.4 123.19)
 		)
 		(stroke
@@
 		)
 	)
-	(label "PWM_A_L"
-		(at 152.4 80.01 0)
+	(label "PWM_A_R"
+		(at 152.4 123.19 0)
 		(effects
 			(font
@@
 	(wire
 		(pts
-			(xy 149.86 123.19) (xy 152.4 123.19)
+			(xy 149.86 125.73) (xy 152.4 125.73)
 		)
 		(stroke
@@
 		)
 	)
-	(label "PWM_B_L"
-		(at 152.4 123.19 0)
+	(label "PWM_B_R"
+		(at 152.4 125.73 0)
 		(effects
 			(font
@@
 	(wire
 		(pts
-			(xy 149.86 125.73) (xy 152.4 125.73)
+			(xy 149.86 163.83) (xy 152.4 163.83)
 		)
 		(stroke
@@
 		)
 	)
-	(label "PWM_A_R"
-		(at 152.4 125.73 0)
+	(label "PWM_B_L"
+		(at 152.4 163.83 0)
 		(effects
 			(font
@@
 	(wire
 		(pts
-			(xy 149.86 163.83) (xy 152.4 163.83)
+			(xy 149.86 113.03) (xy 152.4 113.03)
 		)
 		(stroke
@@
 		)
 	)
-	(label "PWM_B_R"
-		(at 152.4 163.83 0)
+	(label "LED_3"
+		(at 152.4 113.03 0)
 		(effects
 			(font
@@
 	(wire
 		(pts
-			(xy 149.86 113.03) (xy 152.4 113.03)
+			(xy 149.86 115.57) (xy 152.4 115.57)
 		)
 		(stroke
@@
 		)
 	)
-	(label "Enc_A_L"
-		(at 152.4 113.03 0)
+	(label "SW_2"
+		(at 152.4 115.57 0)
 		(effects
 			(font
@@
 	(wire
 		(pts
-			(xy 149.86 115.57) (xy 152.4 115.57)
+			(xy 149.86 156.21) (xy 152.4 156.21)
 		)
 		(stroke
@@
 		)
 	)
-	(label "Enc_B_L"
-		(at 152.4 115.57 0)
+	(label "Enc_A_L"
+		(at 152.4 156.21 0)
 		(effects
 			(font
@@
 	(wire
 		(pts
-			(xy 149.86 156.21) (xy 152.4 156.21)
+			(xy 149.86 158.75) (xy 152.4 158.75)
 		)
 		(stroke
@@
 		)
 	)
-	(label "Enc_A_R"
-		(at 152.4 156.21 0)
+	(label "Enc_B_L"
+		(at 152.4 158.75 0)
 		(effects
 			(font
@@
 	(wire
 		(pts
-			(xy 149.86 158.75) (xy 152.4 158.75)
+			(xy 149.86 120.65) (xy 152.4 120.65)
 		)
 		(stroke
@@
 	)
 	(label "Enc_B_R"
-		(at 152.4 158.75 0)
+		(at 152.4 120.65 0)
 		(effects
 			(font
@@
 	(wire
 		(pts
-			(xy 77.47 128.27) (xy 83.82 128.27)
+			(xy 77.47 148.59) (xy 83.82 148.59)
 		)
 		(stroke
@@
 	)
 	(label "IMU_INT1"
-		(at 77.47 128.27 0)
+		(at 77.47 148.59 0)
 		(effects
 			(font
@@
 	(wire
 		(pts
-			(xy 77.47 130.81) (xy 83.82 130.81)
+			(xy 77.47 151.13) (xy 83.82 151.13)
 		)
 		(stroke
@@
 	)
 	(label "IMU_INT2"
-		(at 77.47 130.81 0)
+		(at 77.47 151.13 0)
 		(effects
 			(font
