File: Robotrace/Robotrace.kicad_sch (KiCad schematic)
At the start: 62 parts, among them J1 USB_C_Receptacle_USB2.0_16P, J10 Side_L, J11 LINE, J6 STDC14, J7 Conn_02x05_Odd_Even, J8 Conn_02x05_Odd_Even, J9 Side_R, Q5 BSS138, U1 STM32F469VGTx, Y1 12MHz

Commit message: 回路図終わり
Parts:
- C1: renamed from C17; footprint Capacitor_SMD:C_0603_1608Metric -> Capacitor_SMD:C_0402_1005Metric
- C10: renamed from C25; footprint Capacitor_SMD:C_0603_1608Metric -> Capacitor_SMD:C_0402_1005Metric
- C11: renamed from C27; footprint Capacitor_SMD:C_0603_1608Metric -> Capacitor_SMD:C_0402_1005Metric
- C12: renamed from C28; footprint Capacitor_SMD:C_0603_1608Metric -> Capacitor_SMD:C_0402_1005Metric
- C13: renamed from C29; footprint Capacitor_SMD:C_0603_1608Metric -> Capacitor_SMD:C_0402_1005Metric
- C14: renamed from C30; footprint Capacitor_SMD:C_0603_1608Metric -> Capacitor_SMD:C_0402_1005Metric
- C15: renamed from C31; footprint Capacitor_SMD:C_0603_1608Metric -> Capacitor_SMD:C_0402_1005Metric
- C16: renamed from C32; footprint Capacitor_SMD:C_0603_1608Metric -> Capacitor_SMD:C_0402_1005Metric
- C17: renamed from C33; footprint Capacitor_SMD:C_0603_1608Metric -> Capacitor_SMD:C_0402_1005Metric
- C18: renamed from C34; footprint Capacitor_SMD:C_0603_1608Metric -> Capacitor_SMD:C_0402_1005Metric
- C19: renamed from C36; value 2.2u -> 4.7
- C2: renamed from C18; footprint Capacitor_SMD:C_0603_1608Metric -> Capacitor_SMD:C_0402_1005Metric
- C20: renamed from C15; footprint Capacitor_SMD:C_0603_1608Metric -> Capacitor_SMD:C_0402_1005Metric
- C21: renamed from C16; footprint Capacitor_SMD:C_0603_1608Metric -> Capacitor_SMD:C_0402_1005Metric
- C22: renamed from C37; footprint Capacitor_SMD:C_0603_1608Metric -> Capacitor_SMD:C_0402_1005Metric
- C23: renamed from C38; footprint Capacitor_SMD:C_0603_1608Metric -> Capacitor_SMD:C_0402_1005Metric
- C24: renamed from C39; footprint Capacitor_SMD:C_0603_1608Metric -> Capacitor_SMD:C_0402_1005Metric
- C25: renamed from C40; footprint Capacitor_SMD:C_0603_1608Metric -> Capacitor_SMD:C_0402_1005Metric
- C4: renamed from C19; footprint Capacitor_SMD:C_0603_1608Metric -> Capacitor_SMD:C_0402_1005Metric
- C5: renamed from C1; footprint Capacitor_SMD:C_0603_1608Metric -> Capacitor_SMD:C_0402_1005Metric
- C7: renamed from C26; footprint Capacitor_SMD:C_0603_1608Metric -> Capacitor_SMD:C_0402_1005Metric
- C9: renamed from C35; footprint Capacitor_SMD:C_0603_1608Metric -> Capacitor_SMD:C_0402_1005Metric
- renumbered C20 to C3, C21 to C6, C24 to C8, D3 to D2, D8 to D3, D9 to D6, D6 to D7, D10 to D8, D11 to D9, J11 to J1, J1 to J2, J9 to J3, J10 to J4, J6 to J5, J7 to J6, J8 to J7, Q5 to Q1, R9 to R1, R7 to R10, R8 to R11, R4 to R2, R11 to R3, R12 to R4, R1 to R5, R2 to R6, R10 to R7, R5 to R8, R6 to R9, S2 to S1, S3 to S2, S1 to S3
Connections:
- net +5V: now also J1.17 (Pin_17)
- net LineSensor1: now also U1.12 (PC0); no longer U1.19 (PA0)
- net LineSensor10: now also U1.27 (PA6); no longer U1.30 (PB1)
- net LineSensor11: now also U1.28 (PA7); no longer U1.12 (PC0)
- net LineSensor12: now also U1.29 (PB0); no longer U1.13 (PC1)
- net LineSensor13: now also U1.30 (PB1); no longer U1.14 (PC2)
- net LineSensor2: now also U1.13 (PC1); no longer U1.20 (PA1)
- net LineSensor3: now also U1.14 (PC2); no longer U1.21 (PA2)
- net LineSensor4: now also U1.19 (PA0); no longer U1.22 (PA3)
- net LineSensor5: now also U1.20 (PA1); no longer U1.25 (PA4)
- net LineSensor6: now also U1.21 (PA2); no longer U1.26 (PA5)
- net LineSensor7: now also U1.22 (PA3); no longer U1.27 (PA6)
- net LineSensor8: now also U1.25 (PA4); no longer U1.28 (PA7)
- net LineSensor9: now also U1.26 (PA5); no longer U1.29 (PB0)
- no-connect marks 27 -> 26
Other:
- sheet DC-DC ports: added V-MCU; removed none

Commit message: 配線終わり
Connections:
- net FLED: now also U1.70 (PA8)
Changed lines of the file:
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@@
+	(wire
+		(pts
+			(xy 149.86 80.01) (xy 152.4 80.01)
+		)
+		(stroke
+			(width 0)
+			(type default)
+		)
+	)
 	(wire
 		(pts
@@
 		(effects
 			(font
+				(size 1.27 1.27)
+			)
+			(justify left bottom)
+		)
+	)
+	(label "FLED"
+		(at 152.4 80.01 0)
+		(effects
+			(font

Commit message: サイドセンサプルアップ追加
Parts:
- added J13, J14: Conn_01x01_Pin, TestPoint:TestPoint_Pad_1.5x1.5mm, symbol Connector:Conn_01x01_Pin
- added Q11: Q_NMOS_SSSGD_AvalancheRated, Package_SO:Vishay_PowerPAK_1212-8_Single, symbol Transistor_FET:Q_NMOS_SSSGD_AvalancheRated
- added R17, R18, R19: 10k, Resistor_SMD:R_0402_1005Metric, symbol Device:R_Small
Connections:
- net +3V3: now also R18.1, R19.1
- net GND: now also Q11.1 (S), Q11.2 (S), Q11.3 (S), R17.2
- net Side_L: now also R19.2
- net Side_R: now also R18.2
- net fan: now reaches U1.53 (PD14)
- net fan: now also Q11.4 (G), R17.1
- new net: J13.1 (Pin_1), Q11.5 (D)
- new net +12V: J14.1 (Pin_1)
Other:
- moved on the sheet: J3, J4

Commit message: メイン基板完成
Connections:
- net +5V: now also J3.2 (Pin_2), J4.2 (Pin_2); no longer J3.3 (Pin_3), J4.3 (Pin_3)
- net PWM_A_L: now also U1.34 (PE9); no longer U1.68 (PC8)
- net PWM_A_R: now also U1.38 (PE13); no longer U1.98 (PB8)
- net PWM_B_L: now also U1.33 (PE8); no longer U1.69 (PC9)
- net PWM_B_R: now also U1.37 (PE12); no longer U1.99 (PB9)
- net Side_L: now also J4.3 (Pin_3); no longer J4.2 (Pin_2)
- net Side_R: now also J3.3 (Pin_3); no longer J3.2 (Pin_2)
Other:
- moved on the sheet: J3, J4

Commit message: 基板完成
Connections:
- net LED_1: now also U1.35 (PE10); no longer U1.80 (PA15)
- net LED_2: now also U1.36 (PE11); no longer U1.31 (PB2)
- net LED_3: now also U1.39 (PE14); no longer U1.93 (PB4)
- net LED_4: now also U1.40 (PE15); no longer U1.41 (PB10)
Changed lines of the file:
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@@
 	(wire
 		(pts
-			(xy 149.86 97.79) (xy 152.4 97.79)
+			(xy 83.82 110.49) (xy 81.28 110.49)
 		)
 		(stroke
@@
 	(wire
 		(pts
-			(xy 149.86 128.27) (xy 152.4 128.27)
+			(xy 83.82 123.19) (xy 81.28 123.19)
 		)
 		(stroke
@@
 	(wire
 		(pts
-			(xy 149.86 107.95) (xy 152.4 107.95)
+			(xy 83.82 113.03) (xy 81.28 113.03)
 		)
 		(stroke
@@
 	(wire
 		(pts
-			(xy 149.86 113.03) (xy 152.4 113.03)
+			(xy 83.82 120.65) (xy 81.28 120.65)
 		)
 		(stroke
@@
 	)
 	(label "LED_4"
-		(at 152.4 128.27 0)
+		(at 81.28 123.19 180)
 		(effects
 			(font
 				(size 1.27 1.27)
 			)
-			(justify left bottom)
+			(justify right bottom)
 		)
 	)
@@
 	)
 	(label "LED_2"
-		(at 152.4 107.95 0)
+		(at 81.28 113.03 180)
 		(effects
 			(font
 				(size 1.27 1.27)
 			)
-			(justify left bottom)
+			(justify right bottom)
 		)
 	)
@@
 	)
 	(label "LED_1"
-		(at 152.4 97.79 0)
+		(at 81.28 110.49 180)
 		(effects
 			(font
 				(size 1.27 1.27)
 			)
-			(justify left bottom)
+			(justify right bottom)
 		)
 	)
@@
 	)
 	(label "LED_3"
-		(at 152.4 113.03 0)
+		(at 81.28 120.65 180)
 		(effects
 			(font
 				(size 1.27 1.27)
 			)
-			(justify left bottom)
+			(justify right bottom)
 		)
 	)
