File: Robotrace/MD.kicad_sch (KiCad schematic)
At the start: 8 parts, among them IC2 MIC4606-2YML-TR, J2 Conn_01x01_Pin, J3 Conn_01x01_Pin, Q1 Q_Dual_NMOS_S1G1S2G2D2D1, Q2 Q_Dual_NMOS_S1G1S2G2D2D1

Commit message: 配線
Parts:
- removed Q1, Q2: Q_Dual_NMOS_S1G1S2G2D2D1, symbol Transistor_FET:Q_Dual_NMOS_S1G1S2G2D2D1
- added Q1, Q3, Q6, Q8: Q_NMOS_SSSGD_AvalancheRated, Package_SO:Vishay_PowerPAK_1212-8_Single, symbol Transistor_FET:Q_NMOS_SSSGD_AvalancheRated
- J2, J3: footprint (none) -> MountingHole:MountingHole_2.2mm_M2_Pad_Via
Connections:
- net +12V: now also Q3.5 (D), Q6.5 (D)
- net AHO: now also Q6.4 (G)
- net AHS: now also Q1.5 (D), Q6.1 (S), Q6.2 (S), Q6.3 (S)
- net ALO: now also Q1.4 (G)
- net BHO: now also Q3.4 (G)
- net BHS: now also Q3.1 (S), Q3.2 (S), Q3.3 (S), Q8.5 (D)
- net BLO: now also Q8.4 (G)
- net GND: now also Q1.1 (S), Q1.2 (S), Q1.3 (S), Q8.1 (S), Q8.2 (S), Q8.3 (S)

Commit message: 回路図終わり
Parts:
- J10: renamed from J3; footprint MountingHole:MountingHole_2.2mm_M2_Pad_Via -> ViaPad:ViaPad_D2.0mm_Drill1.0mm
- J9: renamed from J2; footprint MountingHole:MountingHole_2.2mm_M2_Pad_Via -> ViaPad:ViaPad_D2.0mm_Drill1.0mm
- renumbered C11 to C36, C9 to C37, C10 to C38, Q6 to Q2, Q1 to Q3, Q3 to Q4, Q8 to Q5
