File: Robotrace/Robotrace.kicad_pcb (KiCad board)
At the start: 2 copper layers, 103 parts, among them IC2 MIC4606-2YML-TR, IC3 MIC4606-2YML-TR, J1 USB_C_Receptacle_USB2.0_16P, J10 Side_L, J11 LINE, J12 VIN, J2 Conn_01x01_Pin, J3 Conn_01x01_Pin, J4 Conn_01x01_Pin, J5 Conn_01x01_Pin, J6 STDC14, J7 Conn_02x05_Odd_Even, J8 Conn_02x05_Odd_Even, J9 Side_R, Q1 Q_NMOS_SSSGD_AvalancheRated, Q2 Q_NMOS_SSSGD_AvalancheRated, Q3 Q_NMOS_SSSGD_AvalancheRated, Q4 Q_NMOS_SSSGD_AvalancheRated, Q5 BSS138, Q6 Q_NMOS_SSSGD_AvalancheRated, Q7 Q_NMOS_SSSGD_AvalancheRated, Q8 Q_NMOS_SSSGD_AvalancheRated, Q9 Q_NMOS_SSSGD_AvalancheRated, U1 STM32F469VGTx, U2 TLV70233_SOT23-5, U3 ICM-42688-P, Y1 12MHz

Commit message: 回路図終わり
Parts:
- removed C42: 330u, Capacitor_SMD:CP_Elec_8x6.9
- removed the R3 at (232.0, 67.0)
- added IC1: NJW1933F1-AT-TE2, Package_TO_SOT_SMD:SOT-23-6, B.Cu at (103.3, 106.7)
- added R12: 33k, Resistor_SMD:R_0402_1005Metric, F.Cu at (112.3, 88.9)
- added R13: 10k, Resistor_SMD:R_0402_1005Metric, F.Cu at (112.3, 88.0)
- BZ1, FB1, IC2, IC3, L1, U2: moved to B.Cu
- C1: renamed from C17; footprint Capacitor_SMD:C_0603_1608Metric -> Capacitor_SMD:C_0402_1005Metric
- C10: renamed from C25; footprint Capacitor_SMD:C_0603_1608Metric -> Capacitor_SMD:C_0402_1005Metric
- C11: renamed from C27; footprint Capacitor_SMD:C_0603_1608Metric -> Capacitor_SMD:C_0402_1005Metric
- C12: renamed from C28; footprint Capacitor_SMD:C_0603_1608Metric -> Capacitor_SMD:C_0402_1005Metric; moved to B.Cu
- C13: renamed from C29; footprint Capacitor_SMD:C_0603_1608Metric -> Capacitor_SMD:C_0402_1005Metric; moved to B.Cu
- C14: renamed from C30; footprint Capacitor_SMD:C_0603_1608Metric -> Capacitor_SMD:C_0402_1005Metric
- C15: renamed from C31; footprint Capacitor_SMD:C_0603_1608Metric -> Capacitor_SMD:C_0402_1005Metric
- C16: renamed from C32; footprint Capacitor_SMD:C_0603_1608Metric -> Capacitor_SMD:C_0402_1005Metric
- C17: renamed from C33; footprint Capacitor_SMD:C_0603_1608Metric -> Capacitor_SMD:C_0402_1005Metric
- C18: renamed from C34; footprint Capacitor_SMD:C_0603_1608Metric -> Capacitor_SMD:C_0402_1005Metric
- C19: renamed from C36; value 2.2u -> 4.7
- C2: renamed from C18; footprint Capacitor_SMD:C_0603_1608Metric -> Capacitor_SMD:C_0402_1005Metric
- C20: renamed from C15; footprint Capacitor_SMD:C_0603_1608Metric -> Capacitor_SMD:C_0402_1005Metric; moved to B.Cu
- C21: renamed from C16; footprint Capacitor_SMD:C_0603_1608Metric -> Capacitor_SMD:C_0402_1005Metric; moved to B.Cu
- C22: renamed from C37; footprint Capacitor_SMD:C_0603_1608Metric -> Capacitor_SMD:C_0402_1005Metric
- C23: renamed from C38; footprint Capacitor_SMD:C_0603_1608Metric -> Capacitor_SMD:C_0402_1005Metric
- C24: renamed from C39; footprint Capacitor_SMD:C_0603_1608Metric -> Capacitor_SMD:C_0402_1005Metric
- C25: renamed from C40; footprint Capacitor_SMD:C_0603_1608Metric -> Capacitor_SMD:C_0402_1005Metric
- C27: renamed from C3; footprint Capacitor_SMD:C_0603_1608Metric -> Capacitor_SMD:C_0402_1005Metric; moved to B.Cu
- C28: renamed from C2; moved to B.Cu
- C29: renamed from C22; moved to B.Cu
- C30: renamed from C23; moved to B.Cu
- C31: renamed from C4; moved to B.Cu
- C32: renamed from C5; moved to B.Cu
- C33: renamed from C6; footprint Capacitor_SMD:C_0603_1608Metric -> Capacitor_SMD:C_0402_1005Metric
- C35: renamed from C8; footprint Capacitor_SMD:C_0603_1608Metric -> Capacitor_SMD:C_0402_1005Metric
- C36: renamed from C11; moved to B.Cu
- C37: renamed from C9; moved to B.Cu
- C38: renamed from C10; moved to B.Cu
- C39: renamed from C12; moved to B.Cu
- C4: renamed from C19; footprint Capacitor_SMD:C_0603_1608Metric -> Capacitor_SMD:C_0402_1005Metric
- C40: renamed from C13; moved to B.Cu
- C41: renamed from C14; moved to B.Cu
- C5: renamed from C1; footprint Capacitor_SMD:C_0603_1608Metric -> Capacitor_SMD:C_0402_1005Metric
- C7: renamed from C26; footprint Capacitor_SMD:C_0603_1608Metric -> Capacitor_SMD:C_0402_1005Metric
- C9: renamed from C35; footprint Capacitor_SMD:C_0603_1608Metric -> Capacitor_SMD:C_0402_1005Metric
- D10: renamed from D7; moved to B.Cu
- D11: renamed from D2; moved to B.Cu
- J10: renamed from J3; footprint MountingHole:MountingHole_2.2mm_M2_Pad_Via -> ViaPad:ViaPad_D2.0mm_Drill1.0mm
- J11: renamed from J4; footprint MountingHole:MountingHole_2.2mm_M2_Pad_Via -> ViaPad:ViaPad_D2.0mm_Drill1.0mm
- J12: renamed from J5; footprint MountingHole:MountingHole_2.2mm_M2_Pad_Via -> ViaPad:ViaPad_D2.0mm_Drill1.0mm
- J2: renamed from J1; moved to B.Cu
- J9: renamed from J2; footprint MountingHole:MountingHole_2.2mm_M2_Pad_Via -> ViaPad:ViaPad_D2.0mm_Drill1.0mm
- Q1: renamed from Q5; moved to B.Cu
- Q2: renamed from Q6; moved to B.Cu
- Q4: renamed from Q3; moved to B.Cu
- Q6: renamed from Q7; moved to B.Cu
- Q8: renamed from Q4; moved to B.Cu
- R10: renamed from R7; moved to B.Cu
- R11: renamed from R8; moved to B.Cu
- R14: renamed from R15; moved to B.Cu
- R15: renamed from R16; moved to B.Cu
- R2: renamed from R4; moved to B.Cu
- R3: renamed from R11; moved to B.Cu
- R4: renamed from R12; moved to B.Cu
- R7: renamed from R10; moved to B.Cu
- R8: renamed from R5; moved to B.Cu
- R9: renamed from R6; moved to B.Cu
- moved S5 218.8 mm to (103.0, 107.7), turned to -90 degrees
- moved J8 215.0 mm to (102.8, 90.3)
- moved D3 204.5 mm to (112.2, 101.2)
- moved C26 204.5 mm to (105.7, 98.5), turned to 180 degrees
- moved D6 194.5 mm to (112.1, 103.7)
- moved D8 194.3 mm to (112.1, 106.2)
- moved D9 194.0 mm to (112.1, 108.7)
- moved D2 192.2 mm to (114.9, 83.2)
- moved C23 192.1 mm to (110.0, 103.7), turned to -90 degrees
- moved C24 192.1 mm to (110.0, 106.2), turned to -90 degrees
- moved D4 192.1 mm to (114.9, 84.8)
- moved C25 192.0 mm to (110.0, 108.1), turned to -90 degrees
- moved D5 192.0 mm to (114.9, 86.4)
- moved D7 191.9 mm to (114.9, 88.0)
- moved C22 189.2 mm to (112.5, 99.4)
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- renumbered C41 to C26, C20 to C3, C7 to C34, C21 to C6, C24 to C8, D3 to D2, D8 to D3, D9 to D6, D6 to D7, D10 to D8, D11 to D9, J11 to J1, J9 to J3, J10 to J4, J6 to J5, J7 to J6, J8 to J7, J12 to J8, Q1 to Q3, Q8 to Q5, Q2 to Q7, R9 to R1, R1 to R5, R2 to R6, S2 to S1, S3 to S2, S1 to S3, S6 to S5
Connections:
- J1 pad 17: unconnected-(J11-Pin_17-Pad17) -> +5V
- U1 pad 12: /LineSensor11 -> /LineSensor1
- U1 pad 13: /LineSensor12 -> /LineSensor2
- U1 pad 14: /LineSensor13 -> /LineSensor3
- U1 pad 19: /LineSensor1 -> /LineSensor4
- U1 pad 20: /LineSensor2 -> /LineSensor5
- U1 pad 21: /LineSensor3 -> /LineSensor6
- U1 pad 22: /LineSensor4 -> /LineSensor7
- U1 pad 25: /LineSensor5 -> /LineSensor8
- U1 pad 26: /LineSensor6 -> /LineSensor9
- U1 pad 27: /LineSensor7 -> /LineSensor10
- U1 pad 28: /LineSensor8 -> /LineSensor11
- U1 pad 29: /LineSensor9 -> /LineSensor12
- U1 pad 30: /LineSensor10 -> /LineSensor13
- U1 pad 50: unconnected-(U1-PD8-Pad50) -> /IMU_INT1
- U1 pad 51: unconnected-(U1-PD9-Pad51) -> /IMU_INT2
- U1 pad 66: unconnected-(U1-PC6-Pad66) -> /Enc_A_L
- U1 pad 67: unconnected-(U1-PC7-Pad67) -> /Enc_B_L
- U1 pad 68: /SW_2 -> /PWM_A_L
- U1 pad 69: unconnected-(U1-PC9-Pad69) -> /PWM_B_L
- U1 pad 93: unconnected-(U1-PB4-Pad93) -> /LED_3
- U1 pad 94: unconnected-(U1-PB5-Pad94) -> /SW_2
- U1 pad 95: /LED_3 -> /Enc_A_R
- U1 pad 96: unconnected-(U1-PB7-Pad96) -> /Enc_B_R
- U1 pad 98: unconnected-(U1-PB8-Pad98) -> /PWM_A_R
- U1 pad 99: unconnected-(U1-PB9-Pad99) -> /PWM_B_R
Routing:
- net GND: track 0.00 -> 191.9 mm, vias 0 -> 6
- net +12V: track 0.00 -> 93.5 mm, vias 0 -> 1
- net +3V3: track 0.00 -> 39.5 mm, vias 0 -> 17
- net /RST: track 0.00 -> 37.9 mm, vias 0 -> 3
- net /PWM_B_L: track 0.00 -> 31.7 mm, vias 0 -> 2
- net /PWM_A_L: track 0.00 -> 30.4 mm, vias 0 -> 2
- net /MD_EN: track 0.00 -> 29.5 mm, vias 0 -> 3
- net /D-: track 0.00 -> 27.4 mm, vias 0 -> 2
- net /VCP_TX: track 0.00 -> 25.8 mm, vias 0 -> 2
- net /VCP_RX: track 0.00 -> 25.1 mm, vias 0 -> 2
- net /D+: track 0.00 -> 24.7 mm, vias 0 -> 2
- net /MD/AHS: track 0.00 -> 24.4 mm, vias 0 -> 1
- net /BOOT0: track 0.00 -> 22.9 mm, vias 0 -> 2
- net /MD1/AHS: track 0.00 -> 22.5 mm, vias 0 -> 1
- net /MD1/BHS: track 0.00 -> 22.2 mm, vias 0 -> 1
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- added copper zone on In2.Cu, net +3V3
- added copper zone on In4.Cu, net +5V
- added copper zone on B.Cu, net GND
- added copper zone on F.Cu, net GND
- added copper zone on In1.Cu, net GND
- added copper zone on In3.Cu, net GND
Other:
- board outline added: 50 x 35 mm
- copper layers 2 -> 6

Commit message: 配線終わり
Parts:
- added Q10: SiSS27DN, Package_SO:Vishay_PowerPAK_1212-8_Single, B.Cu at (107.8, 94.7)
- added R16: 10k, Resistor_SMD:R_0402_1005Metric, B.Cu at (105.4, 95.5)
- moved C5 25.3 mm to (134.8, 108.2)
- moved R4 2.19 mm to (114.1, 114.3)
- moved R2 2.18 mm to (110.1, 114.3)
- moved S5 1.81 mm to (104.8, 107.7)
- moved C40 0.28 mm to (139.3, 94.0)
- moved C34 0.06 mm to (116.0, 90.9)
Connections:
- J8 pad 2: +12V -> Net-(J8-Pin_2)
- S5 pad 4: +12V -> /DC-DC/Pch
- S5 pad 5: /DC-DC/EN -> GND
- U1 pad 70: unconnected-(U1-PA8-Pad70) -> /FLED
Routing:
- net /SW_1: track 4.84 -> 38.4 mm, vias 1 -> 2
- net /Enc_B_R: track 0.00 -> 33.5 mm, vias 0 -> 1
- net /Enc_A_R: track 0.00 -> 32.8 mm, vias 0 -> 1
- net /Enc_A_L: track 0.00 -> 32.0 mm, vias 0 -> 1
- net /Enc_B_L: track 0.00 -> 32.0 mm, vias 0 -> 2
- net /LED_1: track 0.00 -> 31.3 mm, vias 0 -> 2
- net /LED_3: track 0.00 -> 27.6 mm, vias 0 -> 2
- net /SW_2: track 4.86 -> 30.8 mm, vias 1 -> 2
- net /IMU_INT2: track 0.00 -> 17.4 mm, vias 0 -> 2
- net /FLED: track 0.00 -> 13.3 mm, vias 0 -> 2
- net /CS: track 0.00 -> 13.3 mm, vias 0 -> 2
- net /IMU_INT1: track 0.00 -> 12.4 mm, vias 0 -> 2
- net /DC-DC/Pch: track 0.00 -> 12.1 mm, vias 0 -> 2
- net /LED_2: track 0.00 -> 11.3 mm, vias 0 -> 2
- net Net-(J2-CC1): track 0.00 -> 11.3 mm, vias 0 -> 1
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- added copper zone on B.Cu, net +12V
- added copper zone on B.Cu, net +5V
- added copper zone on B.Cu, net /MD/AHS
- added copper zone on F.Cu, net /MD/AHS
- added copper zone on B.Cu, net /MD/BHS
- added copper zone on F.Cu, net /MD/BHS
- added copper zone on B.Cu, net /MD1/AHS
- added copper zone on F.Cu, net /MD1/AHS
- added copper zone on B.Cu, net /MD1/BHS
- added copper zone on F.Cu, net /MD1/BHS
- added copper zone on B.Cu, net Net-(J8-Pin_2)

Commit message: サイドセンサプルアップ追加
Parts:
- added J13: Conn_01x01_Pin, TestPoint:TestPoint_Pad_1.5x1.5mm, B.Cu at (118.4, 109.0)
- added J14: Conn_01x01_Pin, TestPoint:TestPoint_Pad_1.5x1.5mm, B.Cu at (118.4, 106.2)
- added Q11: Q_NMOS_SSSGD_AvalancheRated, Package_SO:Vishay_PowerPAK_1212-8_Single, B.Cu at (118.2, 112.7)
- added R17: 10k, Resistor_SMD:R_0402_1005Metric, B.Cu at (117.5, 115.5)
- added R18: 10k, Resistor_SMD:R_0402_1005Metric, F.Cu at (131.1, 110.2)
- added R19: 10k, Resistor_SMD:R_0402_1005Metric, F.Cu at (119.5, 110.0)
Connections:
- U1 pad 53: unconnected-(U1-PD14-Pad53) -> /fan
Routing:
- net /fan: track 0.00 -> 15.8 mm, vias 0 -> 2
- net Net-(J13-Pin_1): track 0.00 -> 3.22 mm
- net +3V3: track 29.4 -> 32.3 mm, vias 21 -> 22
- net /Side_R: track 4.49 -> 7.15 mm
- net /Side_L: track 10.9 -> 12.9 mm
- net GND: vias 126 -> 131
- added copper zone on B.Cu, net Net-(J13-Pin_1)
Other:
- board text added: "+"
- board text added: "-"
- board text added: "BOOT"
- board text added: "RESET"

Commit message: メイン基板完成
Connections:
- J3 pad 2: /Side_R -> +5V
- J3 pad 3: +5V -> /Side_R
- J4 pad 2: /Side_L -> +5V
- J4 pad 3: +5V -> /Side_L
- U1 pad 33: unconnected-(U1-PE8-Pad33) -> /PWM_B_L
- U1 pad 34: unconnected-(U1-PE9-Pad34) -> /PWM_A_L
- U1 pad 37: unconnected-(U1-PE12-Pad37) -> /PWM_B_R
- U1 pad 38: unconnected-(U1-PE13-Pad38) -> /PWM_A_R
- U1 pad 68: /PWM_A_L -> unconnected-(U1-PC8-Pad68)
- U1 pad 69: /PWM_B_L -> unconnected-(U1-PC9-Pad69)
- U1 pad 98: /PWM_A_R -> unconnected-(U1-PB8-Pad98)
- U1 pad 99: /PWM_B_R -> unconnected-(U1-PB9-Pad99)
Routing:
- net /PWM_A_R: track 9.89 -> 24.0 mm
- net /PWM_B_R: track 10.3 -> 23.2 mm
- net /PWM_B_L: track 30.8 -> 22.5 mm
- net /PWM_A_L: track 30.4 -> 22.8 mm
- net /Side_R: track 7.15 -> 5.60 mm
- net GND: vias 131 -> 132

Commit message: 基板完成
Connections:
- U1 pad 31: /LED_2 -> unconnected-(U1-PB2-Pad31)
- U1 pad 35: unconnected-(U1-PE10-Pad35) -> /LED_1
- U1 pad 36: unconnected-(U1-PE11-Pad36) -> /LED_2
- U1 pad 39: unconnected-(U1-PE14-Pad39) -> /LED_3
- U1 pad 40: unconnected-(U1-PE15-Pad40) -> /LED_4
- U1 pad 41: /LED_4 -> unconnected-(U1-PB10-Pad41)
- U1 pad 80: /LED_1 -> unconnected-(U1-PA15-Pad80)
- U1 pad 93: /LED_3 -> unconnected-(U1-PB4-Pad93)
Routing:
- net /LED_1: track 31.3 -> 13.7 mm
- net /LED_3: track 27.6 -> 11.5 mm
- net /LED_2: track 11.3 -> 12.3 mm
- net /LED_4: track 11.2 -> 10.6 mm
- net GND: vias 132 -> 133
Changed lines of the file:
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@@
 	(net 109 "unconnected-(U1-PC8-Pad68)")
 	(net 110 "unconnected-(U1-PD15-Pad54)")
-	(net 111 "unconnected-(U1-PE11-Pad36)")
+	(net 111 "unconnected-(U1-PB2-Pad31)")
 	(net 112 "unconnected-(J5-Pin_10-Pad10)")
 	(net 113 "/LineSensor1")
@@
 	(net 121 "unconnected-(U1-PC9-Pad69)")
 	(net 122 "unconnected-(J6-Pin_4-Pad4)")
-	(net 123 "unconnected-(U1-PE14-Pad39)")
+	(net 123 "unconnected-(U1-PB4-Pad93)")
 	(net 124 "/VBAT_SENSE")
 	(net 125 "unconnected-(U1-DSIHOST_CKP-Pad60)")
 	(net 126 "unconnected-(U1-PD3-Pad87)")
-	(net 127 "unconnected-(U1-PE10-Pad35)")
+	(net 127 "unconnected-(U1-PA15-Pad80)")
 	(net 128 "unconnected-(S5-Pad1)")
 	(net 129 "unconnected-(U1-DSIHOST_D0P-Pad57)")
@@
 	(net 149 "/MISO")
 	(net 150 "/LineSensor9")
-	(net 151 "unconnected-(U1-PE15-Pad40)")
+	(net 151 "unconnected-(U1-PB10-Pad41)")
 	(net 152 "unconnected-(U2-NC-Pad4)")
 	(net 153 "/IMU_INT2")
@@
 			(layers "F.Cu" "F.Mask" "F.Paste")
 			(roundrect_rratio 0.25)
-			(net 87 "/LED_2")
+			(net 111 "unconnected-(U1-PB2-Pad31)")
 			(pinfunction "PB2")
 			(pintype "bidirectional")
@@
 			(layers "F.Cu" "F.Mask" "F.Paste")
 			(roundrect_rratio 0.25)
-			(net 127 "unconnected-(U1-PE10-Pad35)")
+			(net 86 "/LED_1")
 			(pinfunction "PE10")
 			(pintype "bidirectional")
@@
 			(layers "F.Cu" "F.Mask" "F.Paste")
 			(roundrect_rratio 0.25)
-			(net 111 "unconnected-(U1-PE11-Pad36)")
+			(net 87 "/LED_2")
 			(pinfunction "PE11")
 			(pintype "bidirectional")
@@
 			(layers "F.Cu" "F.Mask" "F.Paste")
 			(roundrect_rratio 0.25)
-			(net 123 "unconnected-(U1-PE14-Pad39)")
+			(net 90 "/LED_3")
 			(pinfunction "PE14")
 			(pintype "bidirectional")
@@
 			(layers "F.Cu" "F.Mask" "F.Paste")
 			(roundrect_rratio 0.25)
-			(net 151 "unconnected-(U1-PE15-Pad40)")
+			(net 91 "/LED_4")
 			(pinfunction "PE15")
 			(pintype "bidirectional")
@@
 			(layers "F.Cu" "F.Mask" "F.Paste")
 			(roundrect_rratio 0.25)
-			(net 91 "/LED_4")
+			(net 151 "unconnected-(U1-PB10-Pad41)")
 			(pinfunction "PB10")
 			(pintype "bidirectional")
@@
 			(layers "F.Cu" "F.Mask" "F.Paste")
 			(roundrect_rratio 0.25)
-			(net 86 "/LED_1")
+			(net 127 "unconnected-(U1-PA15-Pad80)")
 			(pinfunction "PA15")
 			(pintype "bidirectional")
@@
 			(layers "F.Cu" "F.Mask" "F.Paste")
 			(roundrect_rratio 0.25)
-			(net 90 "/LED_3")
+			(net 123 "unconnected-(U1-PB4-Pad93)")
 			(pinfunction "PB4")
 			(pintype "bidirectional")
@@
 	)
 	(via
+		(at 136.97 87.75)
+		(size 0.6)
+		(drill 0.3)
+		(layers "F.Cu" "B.Cu")
+		(free yes)
+		(net 4)
+	)
+	(via
 		(at 146.22 104.21)
 		(size 0.45)
@@
 	)
 	(via
-		(at 118.53 93.62)
+		(at 143.55 86.32)
+		(size 0.6)
+		(drill 0.3)
+		(layers "F.Cu" "B.Cu")
+		(free yes)
+		(net 4)
+	)
+	(via
+		(at 118.727 93.98)
 		(size 0.45)
 		(drill 0.2)
@@
 	)
 	(via
-		(at 119.41 92.41)
-		(size 0.45)
-		(drill 0.2)
-		(layers "F.Cu" "B.Cu")
-		(free yes)
-		(net 4)
-	)
-	(via
 		(at 100.24 86.64)
 		(size 0.45)
@@
 	)
 	(segment
-		(start 125.84 107.597108)
-		(end 127.250535 109.007643)
+		(start 119.654 92.879)
+		(end 119.654 93.632932)
+		(width 0.2)
+		(layer "F.Cu")
+		(net 86)
+	)
+	(segment
+		(start 119.135 92.36)
+		(end 119.654 92.879)
 		(width 0.2)
 		(layer "F.Cu")
@@
 	)
 	(segment
-		(start 125.84 107.35)
-		(end 125.84 107.597108)
+		(start 119.654 93.632932)
+		(end 120.285534 94.264466)
 		(width 0.2)
 		(layer "F.Cu")
@@
 	)
 	(via
-		(at 125.84 107.35)
+		(at 119.135 92.36)
 		(size 0.45)
 		(drill 0.2)
@@
 	)
 	(segment
-		(start 121.186 95.0489)
-		(end 125.84 99.7029)
-		(width 0.2)
-		(layer "In3.Cu")
-		(net 86)
-	)
-	(segment
-		(start 116.166 84.582123)
-		(end 116.166 85.5989)
-		(width 0.2)
-		(layer "In3.Cu")
-		(net 86)
-	)
-	(segment
-		(start 125.84 99.7029)
-		(end 125.84 107.35)
+		(start 119.135 87.551123)
+		(end 115.317018 83.733141)
 		(width 0.2)
 		(layer "In3.Cu")
@@
 	)
 	(segment
-		(start 121.186 90.6189)
-		(end 121.186 95.0489)
+		(start 115.317018 83.733141)
+		(end 114.867499 83.733141)
 		(width 0.2)
 		(layer "In3.Cu")
@@
 	)
 	(segment
-		(start 115.317018 83.733141)
-		(end 116.166 84.582123)
+		(start 119.135 92.36)
+		(end 119.135 87.551123)
 		(width 0.2)
 		(layer "In3.Cu")
@@
 	)
 	(segment
-		(start 114.867499 83.733141)
-		(end 115.317018 83.733141)
+		(start 119.253 93.221877)
+		(end 118.61 92.578877)
 		(width 0.2)
-		(layer "In3.Cu")
-		(net 86)
+		(layer "F.Cu")
+		(net 87)
 	)
 	(segment
-		(start 116.166 85.5989)
-		(end 121.186 90.6189)
+		(start 119.253 93.93904)
+		(end 119.253 93.221877)
 		(width 0.2)
-		(layer "In3.Cu")
-		(net 86)
+		(layer "F.Cu")
+		(net 87)
 	)
 	(segment
-		(start 120.66 91.810506)
-		(end 121.699747 92.850253)
+		(start 118.61 92.578877)
+		(end 118.61 91.72)
 		(width 0.2)
 		(layer "F.Cu")
@@
 	)
 	(segment
-		(start 120.66 91.66)
-		(end 120.66 91.810506)
+		(start 119.93198 94.61802)
+		(end 119.253 93.93904)
 		(width 0.2)
 		(layer "F.Cu")
@@
 	)
 	(via
-		(at 120.66 91.66)
+		(at 118.61 91.72)
 		(size 0.45)
 		(drill 0.2)
@@
 	)
 	(segment
-		(start 115.343141 85.343141)
-		(end 120.66 90.66)
+		(start 118.61 88.61)
+		(end 118.61 91.72)
 		(width 0.2)
 		(layer "In3.Cu")
@@
 	)
 	(segment
-		(start 120.66 90.66)
-		(end 120.66 91.66)
+		(start 115.343141 85.343141)
+		(end 118.61 88.61)
 		(width 0.2)
 		(layer "In3.Cu")
@@
 	)
 	(segment
-		(start 125.315 100.37)
-		(end 126.045 101.1)
+		(start 118.201 95.00836)
+		(end 118.201 94.594178)
 		(width 0.2)
 		(layer "F.Cu")
@@
 	)
 	(segment
-		(start 128.53528 101.1)
-		(end 131.846729 104.411449)
-		(width 0.2)
-		(layer "F.Cu")
-		(net 90)
-	)
-	(segment
-		(start 126.045 101.1)
-		(end 128.53528 101.1)
+		(start 118.87132 95.67868)
+		(end 118.201 95.00836)
 		(width 0.2)
 		(layer "F.Cu")
@@
 	)
 	(via
-		(at 125.315 100.37)
+		(at 118.201 94.594178)
 		(size 0.45)
 		(drill 0.2)
@@
 	)
 	(segment
-		(start 125.315 100.37)
-		(end 125.439 100.246)
+		(start 114.89036 86.976)
+		(end 114.867501 86.953141)
 		(width 0.2)
 		(layer "In3.Cu")
@@
 	)
 	(segment
-		(start 125.439 99.869)
-		(end 120.04 94.47)
+		(start 118.202 93.962123)
+		(end 118.077 93.837123)
 		(width 0.2)
 		(layer "In3.Cu")
@@
 	)
 	(segment
-		(start 116.5229 87.09)
-		(end 115.00436 87.09)
+		(start 118.202 94.593178)
+		(end 118.202 93.962123)
 		(width 0.2)
 		(layer "In3.Cu")
@@
 	)
 	(segment
-		(start 120.04 90.6071)
-		(end 116.5229 87.09)
+		(start 118.201 94.594178)
+		(end 118.202 94.593178)
 		(width 0.2)
 		(layer "In3.Cu")
@@
 	)
 	(segment
-		(start 120.04 94.47)
-		(end 120.04 90.6071)
+		(start 115.629877 86.976)
+		(end 114.89036 86.976)
 		(width 0.2)
 		(layer "In3.Cu")
@@
 	)
 	(segment
-		(start 115.00436 87.09)
-		(end 114.867501 86.953141)
+		(start 118.077 89.423123)
+		(end 115.629877 86.976)
 		(width 0.2)
 		(layer "In3.Cu")
@@
 	)
 	(segment
-		(start 125.439 100.246)
-		(end 125.439 99.869)
+		(start 118.077 93.837123)
+		(end 118.077 89.423123)
 		(width 0.2)
 		(layer "In3.Cu")
@@
 	)
 	(segment
-		(start 118.02 94.68)
-		(end 117.574612 95.125388)
+		(start 117.676 94.18)
+		(end 117.676 95.190466)
 		(width 0.2)
 		(layer "F.Cu")
@@
 	)
 	(segment
-		(start 117.574612 95.796186)
-		(end 118.164213 96.385787)
-		(width 0.2)
-		(layer "F.Cu")
-		(net 91)
-	)
-	(segment
-		(start 117.574612 95.125388)
-		(end 117.574612 95.796186)
-		(width 0.2)
-		(layer "F.Cu")
-		(net 91)
-	)
-	(segment
-		(start 118.02 94.46)
-		(end 118.02 94.68)
+		(start 117.676 95.190466)
+		(end 118.517767 96.032233)
 		(width 0.2)
 		(layer "F.Cu")
@@
 	)
 	(via
-		(at 116.52 88.61)
+		(at 117.676 94.18)
 		(size 0.45)
 		(drill 0.2)
@@
 	)
 	(via
-		(at 118.02 94.46)
+		(at 116.52 88.61)
 		(size 0.45)
 		(drill 0.2)
@@
 	(segment
 		(start 116.52 88.61)
-		(end 116.52 89.3158)
-		(width 0.2)
-		(layer "In3.Cu")
-		(net 91)
-	)
-	(segment
-		(start 117.552 93.992)
-		(end 118.02 94.46)
-		(width 0.2)
-		(layer "In3.Cu")
-		(net 91)
-	)
-	(segment
-		(start 117.552 90.3478)
-		(end 117.552 93.992)
+		(end 117.676 89.766)
 		(width 0.2)
 		(layer "In3.Cu")
@@
 	)
 	(segment
-		(start 116.52 89.3158)
-		(end 117.552 90.3478)
+		(start 117.676 89.766)
+		(end 117.676 94.18)
 		(width 0.2)
 		(layer "In3.Cu")
