File: LineBoard/LineBoard.kicad_pcb (KiCad board)
At the start: 2 copper layers, 11 parts, among them IC1 S7136, J1 side_l, Q1 PT17-21B/L41/TR8

Commit message: メイン基板完成
Parts:
- added C1: 0.1u, Capacitor_SMD:C_0603_1608Metric_Pad1.08x0.95mm_HandSolder, B.Cu at (162.1, 105.1)
- added D10: IR17-21C/TR8, LED_SMD:LED_0805_2012Metric, B.Cu at (144.5, 72.0)
- added D11: IR17-21C/TR8, LED_SMD:LED_0805_2012Metric, B.Cu at (150.0, 73.2)
- added D12: IR17-21C/TR8, LED_SMD:LED_0805_2012Metric, B.Cu at (155.4, 74.8)
- added D13: IR17-21C/TR8, LED_SMD:LED_0805_2012Metric, B.Cu at (160.7, 76.6)
- added D14: IR17-21C/TR8, Diode_SMD:D_0805_2012Metric_Pad1.15x1.40mm_HandSolder, B.Cu at (58.0, 60.0)
- added D2: IR17-21C/TR8, LED_SMD:LED_0805_2012Metric, B.Cu at (100.0, 74.8)
- added D3: IR17-21C/TR8, LED_SMD:LED_0805_2012Metric, B.Cu at (105.4, 73.2)
- added D4: IR17-21C/TR8, LED_SMD:LED_0805_2012Metric, B.Cu at (110.9, 72.0)
- added D5: IR17-21C/TR8, LED_SMD:LED_0805_2012Metric, B.Cu at (116.5, 71.1)
- added D6: IR17-21C/TR8, LED_SMD:LED_0805_2012Metric, B.Cu at (122.1, 70.6)
- added D7: IR17-21C/TR8, LED_SMD:LED_0805_2012Metric, B.Cu at (127.7, 70.4)
- added D8: IR17-21C/TR8, LED_SMD:LED_0805_2012Metric, B.Cu at (133.3, 70.6)
- added D9: IR17-21C/TR8, LED_SMD:LED_0805_2012Metric, B.Cu at (138.9, 71.1)
- added IC1: S7136, S7136:DIP575W60P254L560H210Q4N, B.Cu at (157.0, 106.8)
- added J1: side_l, Connector_JST:JST_SH_BM03B-SRSS-TB_1x03-1MP_P1.00mm_Vertical, F.Cu at (138.6, 117.3)
- added J3: Conn_01x18_Pin, 5051101892:CON_5051101892_MOL, F.Cu at (127.8, 85.5)
- added Q10: PT17-21B/L41/TR8, Diode_SMD:D_0805_2012Metric, B.Cu at (109.8, 66.1)
- added Q11: PT17-21B/L41/TR8, Diode_SMD:D_0805_2012Metric, B.Cu at (103.9, 67.4)
- added Q12: PT17-21B/L41/TR8, Diode_SMD:D_0805_2012Metric, B.Cu at (98.2, 69.0)
- added Q13: PT17-21B/L41/TR8, Diode_SMD:D_0805_2012Metric, B.Cu at (92.5, 71.1)
- added Q2: PT17-21B/L41/TR8, Diode_SMD:D_0805_2012Metric, B.Cu at (157.2, 69.0)
- added Q3: PT17-21B/L41/TR8, Diode_SMD:D_0805_2012Metric, B.Cu at (151.5, 67.4)
- added Q4: PT17-21B/L41/TR8, Diode_SMD:D_0805_2012Metric, B.Cu at (145.6, 66.1)
- added Q5: PT17-21B/L41/TR8, Diode_SMD:D_0805_2012Metric, B.Cu at (139.7, 65.2)
- added Q6: PT17-21B/L41/TR8, Diode_SMD:D_0805_2012Metric, B.Cu at (133.7, 64.6)
- added Q7: PT17-21B/L41/TR8, Diode_SMD:D_0805_2012Metric, B.Cu at (127.7, 64.4)
- added Q8: PT17-21B/L41/TR8, Diode_SMD:D_0805_2012Metric, B.Cu at (121.7, 64.6)
- added Q9: PT17-21B/L41/TR8, Diode_SMD:D_0805_2012Metric, B.Cu at (115.7, 65.2)
- added R10: 180, Resistor_SMD:R_0603_1608Metric, F.Cu at (122.1, 70.6)
- added R11: 10k, Resistor_SMD:R_0603_1608Metric, F.Cu at (145.6, 66.1)
- added R12: 10k, Resistor_SMD:R_0603_1608Metric, F.Cu at (139.7, 65.2)
- added R13: 10k, Resistor_SMD:R_0603_1608Metric, F.Cu at (133.7, 64.6)
- added R15: 180, Resistor_SMD:R_0603_1608Metric, F.Cu at (127.7, 70.4)
- added R16: 180, Resistor_SMD:R_0603_1608Metric, F.Cu at (133.3, 70.6)
- added R17: 180, Resistor_SMD:R_0603_1608Metric, F.Cu at (138.9, 71.1)
- added R18: 10k, Resistor_SMD:R_0603_1608Metric, F.Cu at (127.7, 64.4)
- added R19: 10k, Resistor_SMD:R_0603_1608Metric, F.Cu at (121.7, 64.6)
- added R20: 10k, Resistor_SMD:R_0603_1608Metric, F.Cu at (115.7, 65.2)
- added R21: 180, Resistor_SMD:R_0603_1608Metric, F.Cu at (144.5, 72.0)
- added R22: 180, Resistor_SMD:R_0603_1608Metric, F.Cu at (150.0, 73.2)
- added R23: 10k, Resistor_SMD:R_0603_1608Metric, F.Cu at (109.8, 66.1)
- added R24: 10k, Resistor_SMD:R_0603_1608Metric, F.Cu at (103.9, 67.4)
- added R25: 180, Resistor_SMD:R_0603_1608Metric, F.Cu at (155.4, 74.8)
- added R26: 180, Resistor_SMD:R_0603_1608Metric, F.Cu at (160.7, 76.6)
- added R27: 10k, Resistor_SMD:R_0603_1608Metric, F.Cu at (98.2, 69.0)
- added R28: 10k, Resistor_SMD:R_0603_1608Metric, F.Cu at (92.5, 71.1)
- added R3: 180, Resistor_SMD:R_0603_1608Metric, F.Cu at (105.4, 73.2)
- added R6: 10k, Resistor_SMD:R_0603_1608Metric, F.Cu at (157.2, 69.0)
- added R7: 10k, Resistor_SMD:R_0603_1608Metric, F.Cu at (151.5, 67.4)
- added R8: 180, Resistor_SMD:R_0603_1608Metric, F.Cu at (110.9, 72.0)
- added R9: 180, Resistor_SMD:R_0603_1608Metric, F.Cu at (116.5, 71.1)
- C2: renamed from C1; value C_Small -> 0.1u; moved to B.Cu
- D1, Q1: moved to B.Cu
- D15: renamed from D2; moved to B.Cu
- IC2: renamed from IC1; moved to B.Cu
- J2: renamed from J1; footprint Connector_JST:JST_PH_B3B-PH-K_1x03_P2.00mm_Vertical -> Connector_JST:JST_SH_BM03B-SRSS-TB_1x03-1MP_P1.00mm_Vertical
- R14: renamed from R3; footprint Resistor_SMD:R_0603_1608Metric_Pad0.98x0.95mm_HandSolder -> Resistor_SMD:R_0603_1608Metric
- R2: value 10k -> 180
- R4: value 5.6k -> 420; footprint Resistor_SMD:R_0402_1005Metric -> Resistor_SMD:R_0603_1608Metric
- R5: footprint Resistor_SMD:R_0402_1005Metric -> Resistor_SMD:R_0603_1608Metric
- moved Q1 134.2 mm to (162.9, 71.1), turned to -21.3172 degrees
- moved J2 120.5 mm to (118.0, 117.3), turned to 180 degrees
- moved R5 118.0 mm to (162.9, 71.1), turned to 158.683 degrees
- moved IC2 101.0 mm to (104.5, 111.3), turned to 180 degrees
- moved C2 92.7 mm to (94.5, 108.4), turned to 180 degrees
- moved D1 84.5 mm to (94.7, 76.6), turned to -158.683 degrees
- moved R1 81.4 mm to (94.7, 76.6), turned to -158.683 degrees
- moved R2 78.1 mm to (100.0, 74.8), turned to -162.236 degrees
- moved R4 38.9 mm to (58.0, 56.0)
- moved D15 31.6 mm to (64.0, 60.0)
- moved R14 30.5 mm to (64.0, 56.0)
Connections:
- IC2 pad 3: Net-(IC1-VOUT) -> Net-(IC2-VOUT)
- J2 pad 3: Net-(IC1-VOUT) -> Net-(IC2-VOUT)
- Q1 pad 2: /VOUT -> /VOUT1
- R2 pad 1: /VOUT -> +5V
- R2 pad 2: GND -> Net-(D2-A)
- R4 pad 1: +5V -> Net-(D14-A)
- R4 pad 2: Net-(IC1-VOUT) -> +5V
- R5 pad 1: Net-(IC1-VOUT) -> /VOUT1
Routing:
- net /VOUT1: track 0.00 -> 37.9 mm, vias 0 -> 1
- net /VOUT13: track 0.00 -> 37.1 mm, vias 0 -> 1
- net /VOUT2: track 0.00 -> 33.7 mm, vias 0 -> 1
- net /VOUT12: track 0.00 -> 32.9 mm, vias 0 -> 1
- net /VOUT3: track 0.00 -> 29.2 mm, vias 0 -> 1
- net /VOUT11: track 0.00 -> 28.2 mm, vias 0 -> 1
- net /VOUT4: track 0.00 -> 25.5 mm, vias 0 -> 1
- net /VOUT10: track 0.00 -> 24.9 mm, vias 0 -> 1
- net /VOUT5: track 0.00 -> 22.5 mm, vias 0 -> 1
- net /VOUT9: track 0.00 -> 22.3 mm, vias 0 -> 1
- net /VOUT6: track 0.00 -> 20.9 mm, vias 0 -> 1
- net /VOUT8: track 0.00 -> 20.5 mm, vias 0 -> 1
- net /VOUT7: track 0.00 -> 19.0 mm, vias 0 -> 1
- net Net-(D9-A): vias 0 -> 1
- net Net-(D8-A): vias 0 -> 1
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Other:
- board outline added: 123.1 x 70 mm

Commit message: 基板完成
Parts:
- added C3: 0.1u, Capacitor_SMD:C_0603_1608Metric_Pad1.08x0.95mm_HandSolder, F.Cu at (133.0, 81.0)
- added C4: 0.1u, Capacitor_SMD:C_0603_1608Metric_Pad1.08x0.95mm_HandSolder, F.Cu at (123.1, 79.5)
- C1, C2: moved to F.Cu
- R1, R10, R15, R16, R17, R2, R21, R22, R25, R26, R3, R8, R9: moved to B.Cu
- moved R4 96.5 mm to (137.7, 110.3), turned to 180 degrees
- moved D14 94.3 mm to (137.8, 110.3)
- moved R14 76.5 mm to (117.8, 110.3), turned to 180 degrees
- moved D15 73.7 mm to (117.8, 110.3)
- moved C2 25.1 mm to (118.9, 113.9), turned to 0 degrees
- moved C1 24.9 mm to (138.9, 114.0), turned to 0 degrees
- moved IC1 20.4 mm to (137.7, 100.1), turned to 0 degrees
- moved IC2 17.4 mm to (117.9, 100.1), turned to 0 degrees
- moved R21 2.00 mm to (144.9, 70.0)
- moved R8 2.00 mm to (110.5, 70.0)
- moved R22 2.00 mm to (150.5, 71.3)
- moved R3 2.00 mm to (104.9, 71.3)
- moved R26 2.00 mm to (161.4, 74.8)
- moved R1 2.00 mm to (94.0, 74.8)
- moved R15 2.00 mm to (127.7, 68.4)
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Routing:
- net +5V: track 0.00 -> 132.1 mm, vias 0 -> 5
- net +3V3: track 0.00 -> 101.5 mm, vias 0 -> 1
- net GND: track 0.00 -> 94.7 mm, vias 0 -> 227
- net Net-(IC1-VOUT): track 0.00 -> 19.6 mm
- net Net-(IC2-VOUT): track 0.00 -> 19.4 mm
- net Net-(D14-K): track 0.00 -> 9.94 mm
- net Net-(D15-K): track 0.00 -> 9.65 mm
- net /VOUT13: track 37.1 -> 42.2 mm
- net /VOUT11: track 28.2 -> 33.3 mm
- net /VOUT12: track 32.9 -> 37.9 mm
- net /VOUT2: track 33.7 -> 38.6 mm
- net /VOUT1: track 37.9 -> 42.8 mm
- net /VOUT3: track 29.2 -> 34.0 mm
- net /VOUT4: track 25.5 -> 29.4 mm
- net /VOUT10: track 24.9 -> 28.5 mm
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- added copper zone on B.Cu, net GND
- added copper zone on F.Cu, net GND
Other:
- board size 123.1 x 70 mm -> 117 x 70 mm
